File: eagle/AcceleratedLED.brd (EAGLE design)
At the start: 19 parts, among them Q1 16MHZ, U1 ATMEGA328, U8 TXB0108PWR

Commit message: Set pins to things
Parts:
- moved L_LEDS 116.1 mm to (39.6, 30.5), turned to 270 degrees
- moved BLINKERS 112.6 mm to (17.3, 20.3), turned to 90 degrees
- moved C17 102.6 mm to (33.0, 34.5)
- moved R_LEDS 98.1 mm to (39.6, 20.1), turned to 270 degrees
- moved ISP_V13 38.2 mm to (16.3, 27.4), turned to 90 degrees
- moved JP1 11.4 mm to (36.1, 12.4)
- moved S1 7.13 mm to (24.1, 18.0)
- moved C16 6.91 mm to (33.0, 37.1), turned to 0 degrees
- moved C4 4.85 mm to (28.7, 42.2), turned to 90 degrees
- moved C2 3.75 mm to (34.3, 18.5)
- moved R2 3.64 mm to (34.3, 20.8)
- moved C3 2.17 mm to (35.1, 24.9), turned to 90 degrees
- moved Q1 1.14 mm to (35.1, 29.5)
- moved U8 0.72 mm to (26.7, 35.8)
- moved D3 0.25 mm to (20.8, 34.8)
Connections:
- removed net D2: U1.32
- removed net D3: U1.1
- removed net D4: U1.2
- removed net D5: U1.9
- removed net D6: U1.10
- removed net D7: U1.11
- new net L_BLINK: BLINKERS.2, U1.1
- new net L_BO: L_LEDS.2, U1.11
- new net L_DO: L_LEDS.3, U1.10
- new net R_BLINK: BLINKERS.3, U1.32
- new net R_BO: R_LEDS.2, U1.9
- new net R_DO: R_LEDS.3, U1.2
